File: Entwicklung Knoten/Schaltplan/ConnectorHead_RPi.sch (EAGLE design)
At the start: 45 parts, among them IC1 TINY24/44/84-PU, T1 2N7000, T2 2N7000, T3 2N7000, T4 2N7000, T5 2N7000, T8 2N7000

Commit message: Prototypen angepasst - LED Pads vergrößert, um Lösen durch Hebelwirkung zu vermeiden - Pads des Potentiometer vergrößert - Widerstände der Taster angepasst, da es durch leichte Kriechströme zu Verschiebungen kam - Widerstände gegen Masse auf der Sound-Signal, sowie Display-Backlight Leitung hinzugefügt, damit der Floating-Zustand beim Booten des Raspberry Pi's keine ungewollten Effekte auslöst
Parts:
- removed C4: 680µF/16V, rcl:CPOL-EUE3,5-8_FLAT_DOWN
- added C5: 100uF/16V, rcl:CPOL-EUE2.5-6_FLAT_DOWN
- added R19, R20: 10k, rcl:R-EU_0309/V
- R4, R5, R7, R8: value 10k -> 1k
Connections:
- net +3V3: now also R2.2, R6.2; no longer R2.1, R6.1
- net +5V: now also C5.+, R1.2, R3.2; no longer C4.+, R1.1, R3.1
- net DSP_BL: now also R19.1
- net GND: now also C5.-, R19.2, R20.2; no longer C4.-
- net I2C_SCL_3V3: now also R6.1; no longer R6.2
- net I2C_SCL_5V: now also R1.1; no longer R1.2
- net I2C_SDA_3V3: now also R2.1; no longer R2.2
- net I2C_SDA_5V: now also R3.1; no longer R3.2
- net SOUND_SIG: now also R20.1
Other:
- moved on the sheet: D2, IC1, R14, R16, R2, R3, R6, R9, SG1, T3
